Commit message: Adds inertias to double-pendulum

File: models/double-pendulum.urdf.xacro (robot description, xacro)
@@ -2,10 +2,13 @@
   <xacro:property name="depth" value="0.2"/>
   <xacro:property name="pole_radius" value="${depth / 8}"/>
-  <xacro:property name="link_length" value="0.8"/>
+  <xacro:property name="pole_length" value="0.8"/>
+  <xacro:property name="pole_mass" value="0.5"/>
   <xacro:property name="cart_width" value="0.4"/>
   <xacro:property name="cart_height" value="${cart_width / 2}"/>
+  <xacro:property name="cart_mass" value="8.0"/>
   <xacro:property name="elbow_radius" value="${depth / 4}"/>
   <xacro:property name="elbow_depth" value="${pole_radius * 6}"/>
-  <xacro:macro name="link" params="name length radius">
+  <xacro:property name="elbow_mass" value="0.1"/>
+  <xacro:macro name="pole" params="name length radius mass">
     <link name="${name}">
       <visual>
@@ -14,5 +17,13 @@
         </geometry>
       </visual>
+      <inertial>
+	<mass value="${mass}"/>
+	<inertia ixx="${mass * length * length / 3}" ixy="0.0" ixz="0.0"
+		 iyy="0.0" iyz="0.0" izz="${mass * length * length / 3}"/>
+      </inertial>
     </link>
+  </xacro:macro>
+  <xacro:macro name="null_inertia" params="">
+    <inertia ixx="1" ixy="0" ixz="0" iyy="1" iyz="0" izz="1"/>
   </xacro:macro>
   <link name="cart">
@@ -22,7 +33,11 @@
       </geometry>
     </visual>
+    <inertial>
+      <mass value="${cart_mass}"/>
+      <xacro:null_inertia/>
+    </inertial>
   </link>
-  <xacro:link name="link1" length="${link_length}" radius="${pole_radius}"/>
-  <xacro:link name="link2" length="${link_length}" radius="${pole_radius}"/>
+  <xacro:pole name="pole1" length="${pole_length}" radius="${pole_radius}" mass="${pole_mass}"/>
+  <xacro:pole name="pole2" length="${pole_length}" radius="${pole_radius}" mass="${pole_mass}"/>
   <link name="elbow">
     <visual>
@@ -31,22 +46,25 @@
       </geometry>
     </visual>
+    <inertial>
+      <mass value="${elbow_mass}"/>
+      <xacro:null_inertia/>
+    </inertial>
   </link>
-  <joint name="cart_to_link" type="continuous">
+  <joint name="cart_to_pole" type="continuous">
     <axis xyz="0 1 0"/>
     <parent link="cart"/>
-    <child link="link1"/>
-    <origin xyz="0 ${(depth + 2*pole_radius) / 2} ${link_length / 2}"/>
+    <child link="pole1"/>
+    <origin xyz="0 ${(depth + 2*pole_radius) / 2} ${pole_length / 2}"/>
   </joint>
-  <joint name="link_to_elbow" type="fixed">
-    <origin rpy="${pi / 2} 0 0" xyz="0 ${elbow_depth / 3} ${(link_length + elbow_radius) / 2}"/>
-    <parent link="link1"/>
+  <joint name="pole_to_elbow" type="fixed">
+    <origin rpy="${pi / 2} 0 0" xyz="0 ${elbow_depth / 3} ${(pole_length + elbow_radius) / 2}"/>
+    <parent link="pole1"/>
     <child link="elbow"/>
   </joint>
-  <joint name="elbow_to_link" type="continuous">
+  <joint name="elbow_to_pole" type="continuous">
     <axis xyz="0 1 0"/>
-    <!--<origin rpy="-${pi / 2} 0 0" xyz="0 0 ${link_length / 2}"/>-->
-    <origin rpy="${pi/2} 0 0" xyz="0 ${link_length / 2} ${-(elbow_depth/3)}"/>
+    <origin rpy="${pi/2} 0 0" xyz="0 ${pole_length / 2} ${-(elbow_depth/3)}"/>
     <parent link="elbow"/>
-    <child link="link2"/>
+    <child link="pole2"/>
   </joint>
 </robot>
